File: progtomata.kicad_pcb (KiCad board)
At the start: 2 copper layers, 46 parts, among them J1 Conn_01x04_Pin, J2 Conn_01x04_Pin, P1 USB_C_Plug_USB2.0, SW1 SW_SPDT, SW10 SW_Push_LED, SW11 SW_Push_LED, SW12 SW_Push_LED, SW13 SW_Push_LED, SW14 SW_Push_LED, SW15 SW_Push_LED, SW16 SW_Push_LED, SW17 SW_Push_LED, SW2 SW_Push_LED, SW3 SW_Push_LED, SW4 SW_Push_LED, SW5 SW_Push_LED, SW6 SW_Push_LED, SW7 SW_Push_LED, SW8 SW_Push_LED, SW9 SW_Push_LED, U1 STM32F407VGTx, U2 AMS1117-3.3, U3 74LS148, U4 74LS148, Y1 8MHz

Commit message: Update
Parts:
- added D10: SK6812MINI-E, LED_SMD:LED_SK6812MINI-E_3.2x2.8mm_P1.5mm_ReverseMount, F.Cu at (293.5, 123.6)
- added D11: SK6812MINI-E, LED_SMD:LED_SK6812MINI-E_3.2x2.8mm_P1.5mm_ReverseMount, F.Cu at (293.5, 128.5)
- added D12: SK6812MINI-E, LED_SMD:LED_SK6812MINI-E_3.2x2.8mm_P1.5mm_ReverseMount, F.Cu at (293.5, 133.4)
- added D13: SK6812MINI-E, LED_SMD:LED_SK6812MINI-E_3.2x2.8mm_P1.5mm_ReverseMount, F.Cu at (293.5, 138.2)
- added D14: SK6812MINI-E, LED_SMD:LED_SK6812MINI-E_3.2x2.8mm_P1.5mm_ReverseMount, F.Cu at (293.5, 143.1)
- added D15: SK6812MINI-E, LED_SMD:LED_SK6812MINI-E_3.2x2.8mm_P1.5mm_ReverseMount, F.Cu at (301.9, 118.8)
- added D16: SK6812MINI-E, LED_SMD:LED_SK6812MINI-E_3.2x2.8mm_P1.5mm_ReverseMount, F.Cu at (301.9, 123.6)
- added D17: SK6812MINI-E, LED_SMD:LED_SK6812MINI-E_3.2x2.8mm_P1.5mm_ReverseMount, F.Cu at (301.9, 128.5)
- added D18: SK6812MINI-E, LED_SMD:LED_SK6812MINI-E_3.2x2.8mm_P1.5mm_ReverseMount, F.Cu at (301.9, 133.4)
- added D3: SK6812MINI-E, LED_SMD:LED_SK6812MINI-E_3.2x2.8mm_P1.5mm_ReverseMount, F.Cu at (285.1, 118.8)
- added D4: SK6812MINI-E, LED_SMD:LED_SK6812MINI-E_3.2x2.8mm_P1.5mm_ReverseMount, F.Cu at (285.1, 123.6)
- added D5: SK6812MINI-E, LED_SMD:LED_SK6812MINI-E_3.2x2.8mm_P1.5mm_ReverseMount, F.Cu at (285.1, 128.5)
- added D6: SK6812MINI-E, LED_SMD:LED_SK6812MINI-E_3.2x2.8mm_P1.5mm_ReverseMount, F.Cu at (285.1, 133.4)
- added D7: SK6812MINI-E, LED_SMD:LED_SK6812MINI-E_3.2x2.8mm_P1.5mm_ReverseMount, F.Cu at (285.1, 138.2)
- added D8: SK6812MINI-E, LED_SMD:LED_SK6812MINI-E_3.2x2.8mm_P1.5mm_ReverseMount, F.Cu at (285.1, 143.1)
- added D9: SK6812MINI-E, LED_SMD:LED_SK6812MINI-E_3.2x2.8mm_P1.5mm_ReverseMount, F.Cu at (293.5, 118.8)
- C1, C12, C2, C3, C4, C5, C6, C7: footprint Capacitor_SMD:C_0402_1005Metric -> Capacitor_SMD:C_0603_1608Metric
- SW10, SW11, SW12, SW13, SW14, SW15, SW16, SW17, SW2, SW3, SW4, SW5, SW6, SW7, SW8, SW9: value SW_Push_LED -> SW_Push
- moved U1 79.1 mm to (258.9, 88.5)
- moved U2 79.1 mm to (290.4, 70.5)
- moved Y1 79.1 mm to (279.9, 95.0)
- moved U3 79.1 mm to (174.2, 150.1)
- moved U4 79.1 mm to (152.7, 150.3)
- moved C1 79.1 mm to (189.4, 116.8)
- moved C10 79.1 mm to (192.2, 122.7)
- moved C11 79.1 mm to (192.2, 124.6)
- moved C12 79.1 mm to (195.1, 116.8)
- moved C13 79.1 mm to (195.1, 118.7)
- moved C14 79.1 mm to (195.1, 120.7)
- moved C15 79.1 mm to (222.5, 120.0)
- moved C16 79.1 mm to (222.5, 123.1)
- moved C2 79.1 mm to (189.4, 118.7)
- moved C3 79.1 mm to (189.4, 120.7)
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Connections:
- net /SWCLK renamed SWCLK
- net /SWDIO renamed SWDIO
- U1 pad 1: unconnected-(U1-PE2-Pad1) -> ENC1_Q2
- U1 pad 2: unconnected-(U1-PE3-Pad2) -> OLED2_CS
- U1 pad 3: unconnected-(U1-PE4-Pad3) -> OLED2_DC
- U1 pad 38: unconnected-(U1-PE7-Pad38) -> OLED2_SDIN
- U1 pad 4: unconnected-(U1-PE5-Pad4) -> OLED2_RES
- U1 pad 5: unconnected-(U1-PE6-Pad5) -> OLED2_SCLK
- U1 pad 67: ENC1_Q0 -> /LED_DATA_3V3
- U1 pad 68: ENC1_Q1 -> unconnected-(U1-PA9-Pad68)
- U1 pad 77: ENC1_Q2 -> unconnected-(U1-PA15-Pad77)
- U1 pad 95: unconnected-(U1-PB8-Pad95) -> OLED1_SCL
- U1 pad 96: unconnected-(U1-PB9-Pad96) -> OLED1_SDA
- U1 pad 97: unconnected-(U1-PE0-Pad97) -> ENC1_Q0
- U1 pad 98: unconnected-(U1-PE1-Pad98) -> ENC1_Q1
Routing:
- net +5V: track 0.00 -> 70.3 mm, vias 0 -> 8
- net GND: track 0.00 -> 56.0 mm, vias 0 -> 10
- net Net-(D8-DOUT): track 0.00 -> 27.5 mm
- net Net-(D14-DOUT): track 0.00 -> 23.7 mm
- net Net-(D13-DOUT): track 0.00 -> 22.6 mm
- net Net-(D11-DOUT): track 0.00 -> 10.6 mm
- net Net-(D12-DOUT): track 0.00 -> 10.6 mm
- net Net-(D10-DIN): track 0.00 -> 6.87 mm
Other:
- board outline added: 3.6 x 3.2 mm
