File: progtomata.kicad_sch (KiCad schematic)
At the start: 46 parts, among them J1 Conn_01x04_Pin, J2 Conn_01x04_Pin, P1 USB_C_Plug_USB2.0, SW1 SW_SPDT, SW10 SW_Push_LED, SW11 SW_Push_LED, SW12 SW_Push_LED, SW13 SW_Push_LED, SW14 SW_Push_LED, SW15 SW_Push_LED, SW16 SW_Push_LED, SW17 SW_Push_LED, SW2 SW_Push_LED, SW3 SW_Push_LED, SW4 SW_Push_LED, SW5 SW_Push_LED, SW6 SW_Push_LED, SW7 SW_Push_LED, SW8 SW_Push_LED, SW9 SW_Push_LED, U1 STM32F407VGTx, U2 AMS1117-3.3, U3 74LS148, U4 74LS148, Y1 8MHz

Commit message: Update
Parts:
- added C17, C18, C19, C20: 100n, symbol Device:C
- added C33: 100nF, symbol Device:C
- added D3, D4, D5, D6: SK6812MINI-E, LED_SMD:LED_SK6812MINI-E_3.2x2.8mm_P1.5mm_ReverseMount, symbol LED:SK6812MINI-E
- added J3: Conn_01x07_MountingPin, symbol Connector_Generic_MountingPin:Conn_01x07_MountingPin
- added R4: 330, symbol Device:R
- added U5: 74AHCT1G125, symbol 74xGxx:74AHCT1G125
- added U6: SSD1306, symbol SSD1306_OLED-0.91-128x32:SSD1306
- C1, C12, C2, C3, C4, C5, C6, C7: footprint Capacitor_SMD:C_0402_1005Metric -> Capacitor_SMD:C_0603_1608Metric
- SW10, SW11, SW12, SW13, SW14, SW15, SW16, SW17, SW2, SW3, SW4, SW5, SW6, SW7, SW8, SW9: value SW_Push_LED -> SW_Push; symbol Switch:SW_Push_LED -> Switch:SW_Push
Connections:
- net +5V: now also C17.1, C18.1, C19.1, C20.1, C33.1, D3.3 (VDD), D4.3 (VDD), D5.3 (VDD), D6.3 (VDD), J3.7 (Pin_7), U5.5 (VCC)
- net ENC1_Q0: now also U1.97 (PE0); no longer U1.67 (PA8)
- net ENC1_Q1: now also U1.98 (PE1); no longer U1.68 (PA9)
- net ENC1_Q2: now also U1.1 (PE2); no longer U1.77 (PA15)
- net GND: now also C17.2, C18.2, C19.2, C20.2, C33.2, D3.1 (VSS), D4.1 (VSS), D5.1 (VSS), D6.1 (VSS), J3.6 (Pin_6), U5.1, U5.3 (GND)
- net OLED2_CS: now reaches U1.2 (PE3)
- net OLED2_CS: now also J3.1 (Pin_1)
- net OLED2_DC: now reaches U1.3 (PE4)
- net OLED2_DC: now also J3.2 (Pin_2)
- net OLED2_SDIN: now reaches U1.38 (PE7)
- net OLED2_SDIN: now also J3.5 (Pin_5)
- net OLED2_RES: now reaches U1.4 (PE5)
- net OLED2_RES: now also J3.3 (Pin_3)
- net OLED2_SCLK: now reaches U1.5 (PE6)
- net OLED2_SCLK: now also J3.4 (Pin_4)
- net OLED1_SCL: now reaches U1.95 (PB8)
- net OLED1_SDA: now reaches U1.96 (PB9)
- new net: D3.2 (DIN), R4.1
- new net: D3.4 (DOUT), D4.2 (DIN)
- new net: D4.4 (DOUT), D5.2 (DIN)
- new net: D5.4 (DOUT), D6.2 (DIN)
- new net LED_DATA: R4.2, U5.4
- new net LED_DATA_3V3: U1.67 (PA8), U5.2
- new net LED_I1: D6.4 (DOUT)
- no-connect marks 111 -> 85
Other:
- note added: "Arrows"
- note added: "FX Interface"
- note added: "Priority encoder"
- note added: "Step/ notes"
- note removed: "Buttons priority encoder (sample & steps)"
- note removed: "Interface buttons (audio samples & steps)"
- moved on the sheet: C10, C11, C13, C14, C15, C16, C8, C9, D1, FB1, J1, J2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
